File: iCEBrainstorm/iCEBrainstorm.kicad_sch (KiCad schematic)
At the start: 85 parts, among them J1 Connector, USB-TYPE-C-16P, J2 Conn_01x06_Pin, J3 Connector, USB-TYPE-C-16P, J5 Conn_01x06_Pin, Q1 HL2312, SW1 SW_DIP_x08, SW2 SW_DIP_x08, U1 AMS1117-3.3, U2 AMS1117-1.2, U3 STM32F412RETx, U4 ICE40UP5K-SG48ITR, U5 W25Q128, X1 16 MHz

Commit message: finalised the schematic
Parts:
- added C29, C30, C31, C32: 1uF, PCM_JLCPCB:C_0603, symbol PCM_JLCPCB-Capacitors:0603,1uF
- added D1, D10, D11, D12, D13, D6, D7, D8, D9: Green, PCM_JLCPCB:D_0805, symbol PCM_JLCPCB-Diodes:LED,0805,Green
- added J10, J6, J9: Conn_01x02_Pin, Connector_PinHeader_1.27mm:PinHeader_1x02_P1.27mm_Vertical, symbol Connector:Conn_01x02_Pin
- added J4: Conn_01x16_Pin, Connector_PinHeader_1.27mm:PinHeader_1x16_P1.27mm_Vertical, symbol Connector:Conn_01x16_Pin
- added J7, J8: Conn_01x03_Pin, Connector_PinHeader_1.27mm:PinHeader_1x03_P1.27mm_Vertical, symbol Connector:Conn_01x03_Pin
- added R24, R25, R26, R27, R28, R29, R30, R31, R56, R58, R60, R62: 15kΩ, PCM_JLCPCB:R_0603, symbol PCM_JLCPCB-Resistors:0603,15kΩ
- added R32, R33, R34, R35, R36, R37, R38, R39, R40, R57, R59, R61, R63: 1.5kΩ, PCM_JLCPCB:R_0603, symbol PCM_JLCPCB-Resistors:0603,1.5kΩ
- added S3, S4, S5, S6: RESET, PCM_JLCPCB:SW-SMD_4P-L5.1-W5.1-P3.70-LS6.5-TL-2, symbol PCM_JLCPCB-Connectors_Buttons:Tactile Button, 160gf, 12V, 50mA, 5.1mm
- JP2, JP3, JP4, JP5: footprint (none) -> Jumper:SolderJumper-2_P1.3mm_Bridged_RoundedPad1.0x1.5mm
- JP6, JP7, JP8, JP9: footprint (none) -> Jumper:SolderJumper-2_P1.3mm_Open_RoundedPad1.0x1.5mm
Connections:
- net FPGA_GLOBAL_0 is gone; now on net FPGA_CLK: U3.29 (PB10), U4.35 (IOT_46b_G0)
- net SWDO is gone; now on net SWO: J2.4 (Pin_4)
- net USB_ID is gone; now on net USART1_RX: U3.43 (PA10)
- net USB_SOF is gone; now on net FPGA_GLOBAL_1: U3.41 (PA8)
- net USB_VBUS is gone; now on net USART1_TX: U3.42 (PA9)
- net +3V3: now also SW2.10, SW2.11, SW2.12, SW2.13, SW2.14, SW2.15, SW2.16, SW2.9, J4.10 (Pin_10), R57.1, R59.1, R61.1, R63.1
- net FPGA_CLK: no longer U4.20 (IOB_25b_G3)
- net FPGA_GLOBAL_6: now also J10.2 (Pin_2)
- net GND: now also C29.2, C30.2, C31.2, C32.2, R24.1, R25.1, R26.1, R27.1, R28.1, R29.1, R30.1, R31.1, R32.2, R33.2, R34.2, R35.2, R36.2, R37.2, R38.2, R39.2, R40.2, R56.1, R58.1, R60.1, R62.1
- net FUD-: now reaches R18.2, U4.13 (IOB_24a)
- net IN0: now reaches SW2.1
- net IN0: now also U3.14 (PA0), R24.2
- net IN1: now reaches SW2.2
- net IN1: now also U3.15 (PA1), R25.2
- net IN2: now reaches SW2.3
- net IN2: now also R26.2
- net IN3: now reaches SW2.4
- net IN3: now also U3.56 (PB4), R27.2
- net IN4: now reaches SW2.5
- net IN4: now also U4.10 (IOB_18a), R28.2
- net IN5: now reaches SW2.6
- net IN5: now also U4.11 (IOB_20a), R29.2
- net IN6: now reaches SW2.7
- net IN6: now also U4.6 (IOB_13b), R30.2
- net IN7: now reaches SW2.8
- net IN7: now also U4.4 (IOB_8a), R31.2
- net OUT1: now reaches U4.2 (IOB_6a)
- net OUT1: now also D6.2
- net OUT0: now reaches U4.3 (IOB_9b)
- net OUT0: now also D1.2
- net OUT5: now reaches U4.45 (IOB_5b)
- net OUT5: now also D10.2
- net OUT4: now reaches U4.46 (IOB_0a)
- net OUT4: now also D9.2
- net OUT3: now reaches U4.47 (IOB_2a)
- net OUT3: now also D8.2
- net OUT2: now reaches U4.48 (IOB_4a)
- net OUT2: now also D7.2
- net I2C1_SDA: now reaches U4.18 (IOB_31b)
- net I2C1_SDA: now also U3.59 (PB7), J6.2 (Pin_2)
- net I2C1_SCL: now reaches U4.19 (IOB_29b)
- net I2C1_SCL: now also U3.58 (PB6), J6.1 (Pin_1)
- net FUD+: now reaches R17.2, U4.21 (IOB_23b)
- net PC2: now reaches U3.10 (PC2)
- net PC2: now also J4.3 (Pin_3)
- net PC3: now reaches U3.11 (PC3)
- net PC3: now also J4.4 (Pin_4)
- net USART2_TX: now reaches U3.16 (PA2)
- net USART2_TX: now also J9.1 (Pin_1)
- net USART2_RX: now reaches U3.17 (PA3)
- net USART2_RX: now also J9.2 (Pin_2)
- net PC13: now reaches U3.2 (PC13)
- net PC13: now also J4.14 (Pin_14)
- net SPI1_SCK: now reaches JP7.1 (A), U3.21 (PA5)
- net SPI1_MISO: now reaches JP8.1 (A), U3.22 (PA6)
- net SPI1_MOSI: now reaches JP9.1 (A), U3.23 (PA7)
- net PC4: now reaches U3.24 (PC4)
- net PC4: now also J4.5 (Pin_5)
- net PC5: now reaches U3.25 (PC5)
- net PC5: now also J4.6 (Pin_6)
- net I2S5_CK: now reaches U3.26 (PB0)
- net I2S5_CK: now also J7.1 (Pin_1)
- net I2S5_WS: now reaches U3.27 (PB1)
- net I2S5_WS: now also J7.2 (Pin_2)
- net PC14: now reaches U3.3 (PC14)
- net PC14: now also J4.15 (Pin_15)
- net PC6: now reaches U3.37 (PC6)
- net PC6: now also J4.7 (Pin_7)
- net PC7: now reaches U3.38 (PC7)
- net PC7: now also J4.8 (Pin_8)
- net PC8: now reaches U3.39 (PC8)
- net PC8: now also J4.9 (Pin_9)
- net PC15: now reaches U3.4 (PC15)
- net PC15: now also J4.16 (Pin_16)
- net FPGA_BUS0: now reaches U3.50 (PA15)
- net FPGA_BUS0: now also U4.23 (IOT_37a)
- net PC10: now reaches U3.51 (PC10)
- net PC10: now also J4.11 (Pin_11)
- net PC11: now reaches U3.52 (PC11)
- net PC11: now also J4.12 (Pin_12)
- net PC12: now reaches U3.53 (PC12)
- net PC12: now also J4.13 (Pin_13)
- net FPGA_BUS1: now reaches U3.54 (PD2)
- net FPGA_BUS1: now also U4.25 (IOT_36b)
- net OUT8: now reaches U3.57 (PB5)
- net OUT8: now also D13.2
- net I2S5_SD: now reaches U3.61 (PB8)
- net I2S5_SD: now also J7.3 (Pin_3)
- net BTN0: now reaches U3.62 (PB9)
- net BTN0: now also C30.1, R58.2, S4.4 (D)
- net PC0: now reaches U3.8 (PC0)
- net PC0: now also J4.1 (Pin_1)
- net PC1: now reaches U3.9 (PC1)
- net PC1: now also J4.2 (Pin_2)
- net USART1_RX: now reaches U4.26 (IOT_39a)
- net USART1_TX: now reaches U4.27 (IOT_38b)
- net BTN1: now reaches U4.36 (IOT_48b)
- net BTN1: now also C29.1, R56.2, S3.4 (D)
- net BTN2: now reaches U4.38 (IOT_50b)
- net BTN2: now also C31.1, R60.2, S5.4 (D)
- net RGB0: now reaches U4.39 (RGB0)
- net RGB0: now also J8.1 (Pin_1)
- net RGB1: now reaches U4.40 (RGB1)
- net RGB1: now also J8.2 (Pin_2)
- net RGB2: now reaches U4.41 (RGB2)
- net RGB2: now also J8.3 (Pin_3)
- net OUT7: now reaches U4.42 (IOT_51a)
- net OUT7: now also D12.2
- net OUT6: now reaches U4.43 (IOT_49a)
- net OUT6: now also D11.2
- new net: R59.2, S4.2 (B)
- new net: D6.1, R33.1
- new net: D9.1, R36.1
- new net: R57.2, S3.2 (B)
- new net: D11.1, R38.1
- new net: R63.2, S6.2 (B)
- new net: R61.2, S5.2 (B)
- new net: D1.1, R32.1
- new net: D8.1, R35.1
- new net: D10.1, R37.1
- new net: D13.1, R40.1
- new net: D7.1, R34.1
- new net: D12.1, R39.1
- new net BTN3: C32.1, R62.2, S6.4 (D)
- new net FPGA_GLOBAL_3: J10.1 (Pin_1), U4.20 (IOB_25b_G3)
- no-connect marks 8 -> 28
Other:
- note added: "FPGA_GLOBAL"
- note added: "FPGA_RGB"
- note added: "GPIO"
- note added: "I2C"
- note added: "I2S"
- note added: "IO Headers"
- note added: "USART"
- moved on the sheet: C10, C22, C23, C24, C25, C26, C27, C28, D5, J5, JP2, JP3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

Commit message: still checking schematic
Parts:
- removed C31, C32: 1uF, PCM_JLCPCB:C_0603, symbol PCM_JLCPCB-Capacitors:0603,1uF
- removed R60, R62: 15kΩ, PCM_JLCPCB:R_0603, symbol PCM_JLCPCB-Resistors:0603,15kΩ
- removed R61, R63: 1.5kΩ, PCM_JLCPCB:R_0603, symbol PCM_JLCPCB-Resistors:0603,1.5kΩ
- removed S5, S6: RESET, PCM_JLCPCB:SW-SMD_4P-L5.1-W5.1-P3.70-LS6.5-TL-2, symbol PCM_JLCPCB-Connectors_Buttons:Tactile Button, 160gf, 12V, 50mA, 5.1mm
- added J4, J5: Conn_01x08_Pin, Connector_PinHeader_1.27mm:PinHeader_1x08_P1.27mm_Vertical, symbol Connector:Conn_01x08_Pin
- added JP12, JP13, JP6, JP7: SolderJumper_2_Open, Jumper:SolderJumper-2_P1.3mm_Open_RoundedPad1.0x1.5mm, symbol Jumper:SolderJumper_2_Open
- added R24, R40, R42: 1.5kΩ, PCM_JLCPCB:R_0603, symbol PCM_JLCPCB-Resistors:0603,1.5kΩ
- renumbered C4 to C1, C11 to C10, C14 to C11, C15 to C12, C16 to C13, C17 to C14, C18 to C15, C19 to C16, C9 to C17, C20 to C18, C21 to C19, C5 to C2, C13 to C20, C10 to C21, C24 to C22, C22 to C23, C23 to C24, C30 to C26, C26 to C28, C27 to C29, C7 to C3, C28 to C30, C29 to C32, C8 to C4, C2 to C5, C3 to C6, C1 to C7, C12 to C8, C6 to C9, D2 to D1, D3 to D2, D4 to D3, D5 to D4, D1 to D5, J9 to J10, J5 to J11, J3 to J12, J4 to J3, J7 to J6, J8 to J7, J10 to J8, J6 to J9, JP4 to JP10, JP5 to JP11, JP6 to JP2, JP7 to JP3, JP8 to JP4, JP9 to JP5, JP2 to JP8, JP3 to JP9, R8 to R1, R22 to R10, R6 to R11, R7 to R12, R23 to R14, R18 to R15, R24 to R16, R25 to R17, R26 to R18, R27 to R19, R9 to R2, R28 to R20, R29 to R21, R30 to R22, R31 to R23, R16 to R25, R17 to R26, R12 to R27, R21 to R28, R32 to R29, R33 to R30, R34 to R31, R35 to R32, R36 to R33, R37 to R34, R38 to R35, R39 to R36, R40 to R37, R19 to R38, R58 to R39, R59 to R41, R20 to R43, R56 to R45, R57 to R47, R14 to R48, R15 to R49, R10 to R5, R11 to R6, R5 to R7, R1 to R8, R2 to R9, S2 to S1, S1 to S2, S4 to S3, S3 to S6
Connections:
- net BTN2 is gone; now on net BTN1: U4.38 (IOT_50b)
- net IN4 is gone; now on net FPGA_CLK: R20.2, SW2.5, U4.10 (IOB_18a)
- net SPI2_NSS is gone; now on net IN5: U3.33 (PB12), U4.34 (IOT_44b)
- net +3V3: now also R40.1, R42.1
- net BTN0: now also U4.36 (IOT_48b); no longer U3.62 (PB9)
- net BTN1: no longer U4.36 (IOT_48b)
- net FPGA_CLK: now also J5.5 (Pin_5)
- net FPGA_SPI_SI: now also JP4.2 (B); no longer JP5.2 (B)
- net FPGA_SPI_SO: now also JP5.2 (B); no longer JP4.2 (B)
- net FUD-: now also R24.2
- net GND: now also SW1.10, SW1.11, SW1.12, SW1.9, JP12.1 (A), JP13.1 (A), JP6.1 (A), JP7.1 (A); no longer R16.1, R17.1, R18.1, R19.1, R20.1, R21.1, R22.1, R23.1, R29.2, R30.2, R31.2, R32.2, R33.2, R34.2, R35.2, R36.2
- net I2C1_SCL: now also R42.2
- net I2C1_SDA: now also R40.2
- net IN0: now also J5.1 (Pin_1)
- net IN1: now also J5.2 (Pin_2)
- net IN2: now also U3.56 (PB4), J5.3 (Pin_3)
- net IN3: now also U3.62 (PB9), J5.4 (Pin_4); no longer U3.56 (PB4)
- net IN5: now also J5.6 (Pin_6)
- net IN6: now also J5.7 (Pin_7)
- net IN7: now also J5.8 (Pin_8)
- net OUT0: now also J4.1 (Pin_1)
- net OUT1: now also J4.2 (Pin_2)
- net OUT2: now also J4.3 (Pin_3)
- net OUT3: now also J4.4 (Pin_4)
- net OUT4: now also J4.5 (Pin_5)
- net OUT5: now also J4.6 (Pin_6)
- net OUT6: now also J4.7 (Pin_7)
- net OUT7: now also J4.8 (Pin_8)
- net IN_GND0: now reaches SW1.5
- net IN_GND0: now also R16.1, R17.1, R18.1, R19.1, JP6.2 (B)
- net IN_GND1: now reaches SW1.6
- net IN_GND1: now also R20.1, R21.1, R22.1, R23.1, JP7.2 (B)
- net LED_GND0: now reaches SW1.7
- net LED_GND0: now also R29.2, R30.2, R31.2, R32.2, JP12.2 (B)
- net LED_GND1: now reaches SW1.8
- net LED_GND1: now also R33.2, R34.2, R35.2, R36.2, JP13.2 (B)
- net at R25.1, U4.12 (IOB_22a): now also R24.1
- no-connect marks 28 -> 16
Other:
- note added: "SW1 OFF: Custom Boot SW1 ON: STM Bootloader SW2 OFF: System Memory (default) SW2 ON: Embedded SRAM Boot SW3 OFF: FPGA Custom Boot SW3 ON: FPGA USB DFU Programmer SW4 OFF: FPGA Boot from Flash SW4 ON: FPGA Boot from SPI SW5 OFF: Enable IN0 SW5 ON: Disable IN0 SW6 OFF: Enable IN1 SW6 ON: Disable IN1 SW7 OFF: Enable OUT0 SW7 ON: Disable OUT0 SW8 OFF: Enable OUT1 SW8 ON: Disable OUT1"
- note added: "just make a place for 2, if there are any mistakes"
- note removed: "SW1 OFF: Custom Boot SW1 ON: STM Bootloader SW2 OFF: System Memory (default) SW2 ON: Embedded SRAM Boot SW3 OFF: FPGA Custom Boot SW3 ON: FPGA USB DFU Programmer SW4 OFF: FPGA Boot from Flash SW4 ON: FPGA Boot from SPI"
- note removed: "TODO: is this correct? D+ or D- ??"
- moved on the sheet: D13, R15, R37

Commit message: did some placment
Parts:
- added C26, C27: 100nF, PCM_JLCPCB:C_0603, symbol PCM_JLCPCB-Capacitors:0603,100nF
- J10, J8, J9: footprint Connector_PinHeader_1.27mm:PinHeader_1x02_P1.27mm_Vertical -> Connector_PinHeader_2.54mm:PinHeader_1x02_P2.54mm_Vertical
- J11, J2: footprint Connector_PinHeader_1.27mm:PinHeader_1x06_P1.27mm_Vertical -> Connector_PinHeader_2.54mm:PinHeader_1x06_P2.54mm_Vertical
- J3: footprint Connector_PinHeader_1.27mm:PinHeader_1x16_P1.27mm_Vertical -> Connector_PinHeader_2.54mm:PinHeader_1x16_P2.54mm_Vertical
- J4, J5: footprint Connector_PinHeader_1.27mm:PinHeader_1x08_P1.27mm_Vertical -> Connector_PinHeader_2.54mm:PinHeader_1x08_P2.54mm_Vertical
- J6, J7: footprint Connector_PinHeader_1.27mm:PinHeader_1x03_P1.27mm_Vertical -> Connector_PinHeader_2.54mm:PinHeader_1x03_P2.54mm_Vertical
- renumbered C26 to C28, C28 to C29, C29 to C30, C30 to C31, R40 to R15, R42 to R16, R15 to R17, R16 to R18, R17 to R19, R18 to R20, R19 to R21, R20 to R22, R21 to R23, R22 to R24, R23 to R25, R24 to R26, R25 to R27, R26 to R28, R27 to R29, R28 to R30, R29 to R31, R30 to R32, R31 to R33, R32 to R34, R33 to R35, R34 to R36, R35 to R37, R36 to R38, R37 to R39, R38 to R40, R39 to R41, R41 to R42, R45 to R44, R47 to R45, R48 to R46, R49 to R47, S6 to S4
Connections:
- net +1V2: now also C26.1, C27.1
- net FPGA_CLK: no longer J5.5 (Pin_5), R22.2, SW2.5, U4.10 (IOB_18a)
- net GND: now also C26.2, C27.2
- net IN5: no longer U3.33 (PB12), U4.34 (IOT_44b)
- new net IN4: J5.5 (Pin_5), R22.2, SW2.5, U4.10 (IOB_18a)
- new net SPI2_NSS: U3.33 (PB12), U4.34 (IOT_44b)
