File: iCEBrainstorm/iCEBrainstorm.kicad_pcb (KiCad board)
At the start: 2 copper layers, 70 x 70 mm, 133 parts, among them J1 Connector, USB-TYPE-C-16P, J10 Conn_01x02_Pin, J2 Conn_01x06_Pin, J3 Connector, USB-TYPE-C-16P, J4 Conn_01x16_Pin, J5 Conn_01x06_Pin, J6 Conn_01x02_Pin, J7 Conn_01x03_Pin, J8 Conn_01x03_Pin, J9 Conn_01x02_Pin, Q1 HL2312, SW1 SW_DIP_x08, SW2 SW_DIP_x08, U1 AMS1117-3.3, U2 AMS1117-1.2, U3 STM32F412RETx, U4 ICE40UP5K-SG48ITR, U5 W25Q128, X1 16 MHz

Commit message: still checking schematic
Parts:
- removed C31: 1uF, PCM_JLCPCB:C_0603
- removed the C32 at (205.6, 161.6)
- removed R60, R62: 15kΩ, PCM_JLCPCB:R_0603
- removed R61, R63: 1.5kΩ, PCM_JLCPCB:R_0603
- removed S5: RESET, PCM_JLCPCB:SW-SMD_4P-L5.1-W5.1-P3.70-LS6.5-TL-2
- removed the S6 at (199.6, 161.6)
- added J4: Conn_01x08_Pin, Connector_PinHeader_1.27mm:PinHeader_1x08_P1.27mm_Vertical, F.Cu at (185.8, 111.3)
- added J5: Conn_01x08_Pin, Connector_PinHeader_1.27mm:PinHeader_1x08_P1.27mm_Vertical, F.Cu at (165.0, 110.6)
- added JP12: SolderJumper_2_Open, Jumper:SolderJumper-2_P1.3mm_Open_RoundedPad1.0x1.5mm, F.Cu at (201.7, 114.5)
- added JP13: SolderJumper_2_Open, Jumper:SolderJumper-2_P1.3mm_Open_RoundedPad1.0x1.5mm, F.Cu at (201.5, 99.0)
- added JP6: SolderJumper_2_Open, Jumper:SolderJumper-2_P1.3mm_Open_RoundedPad1.0x1.5mm, F.Cu at (175.3, 107.5)
- added JP7: SolderJumper_2_Open, Jumper:SolderJumper-2_P1.3mm_Open_RoundedPad1.0x1.5mm, F.Cu at (175.2, 94.5)
- added R24: 1.5kΩ, PCM_JLCPCB:R_0603, F.Cu at (106.5, 82.5)
- added R40: 1.5kΩ, PCM_JLCPCB:R_0603, F.Cu at (96.0, 142.8)
- added R42: 1.5kΩ, PCM_JLCPCB:R_0603, F.Cu at (96.0, 145.0)
- moved C10 44.6 mm to (42.2, 138.5)
- moved S1 44.6 mm to (36.2, 138.2)
- moved C21 43.1 mm to (145.5, 151.3)
- moved S2 43.1 mm to (151.2, 150.4)
- moved R10 16.0 mm to (36.0, 98.9)
- moved R11 16.0 mm to (49.8, 93.2)
- moved R12 16.0 mm to (49.5, 95.7)
- moved R13 16.0 mm to (50.1, 98.4)
- moved R14 16.0 mm to (50.1, 101.2)
- moved R8 16.0 mm to (36.5, 93.2)
- moved R9 16.0 mm to (36.8, 95.4)
- moved SW1 16.0 mm to (39.4, 93.3)
- moved D11 13.1 mm to (192.0, 99.3)
- moved D13 13.1 mm to (192.1, 120.7)
- moved D5 13.1 mm to (192.0, 117.7)
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- renumbered C4 to C1, C11 to C10, C14 to C11, C15 to C12, C16 to C13, C17 to C14, C18 to C15, C19 to C16, C9 to C17, C20 to C18, C21 to C19, C5 to C2, C13 to C20, C10 to C21, C24 to C22, C22 to C23, C23 to C24, C30 to C26, C26 to C28, C27 to C29, C7 to C3, C28 to C30, C29 to C32, C8 to C4, C2 to C5, C3 to C6, C1 to C7, C12 to C8, C6 to C9, D2 to D1, D3 to D2, D4 to D3, D5 to D4, D1 to D5, J9 to J10, J5 to J11, J3 to J12, J4 to J3, J7 to J6, J8 to J7, J10 to J8, J6 to J9, JP4 to JP10, JP5 to JP11, JP6 to JP2, JP7 to JP3, JP8 to JP4, JP9 to JP5, JP2 to JP8, JP3 to JP9, R8 to R1, R22 to R10, R6 to R11, R7 to R12, R23 to R14, R18 to R15, R24 to R16, R25 to R17, R26 to R18, R27 to R19, R9 to R2, R28 to R20, R29 to R21, R30 to R22, R31 to R23, R16 to R25, R17 to R26, R12 to R27, R21 to R28, R32 to R29, R33 to R30, R34 to R31, R35 to R32, R36 to R33, R37 to R34, R38 to R35, R39 to R36, R40 to R37, R19 to R38, R58 to R39, R59 to R41, R20 to R43, R56 to R45, R57 to R47, R14 to R48, R15 to R49, R10 to R5, R11 to R6, R5 to R7, R1 to R8, R2 to R9, S2 to S1, S1 to S2, S4 to S3, S3 to S6
Connections:
- R16 pad 1: GND -> /IN_GND0
- R17 pad 1: GND -> /IN_GND0
- R18 pad 1: GND -> /IN_GND0
- R19 pad 1: GND -> /IN_GND0
- R20 pad 1: GND -> /IN_GND1
- R20 pad 2: /IN4 -> /FPGA_CLK
- R21 pad 1: GND -> /IN_GND1
- R22 pad 1: GND -> /IN_GND1
- R23 pad 1: GND -> /IN_GND1
- R29 pad 2: GND -> /LED_GND0
- R30 pad 2: GND -> /LED_GND0
- R31 pad 2: GND -> /LED_GND0
- R32 pad 2: GND -> /LED_GND0
- R33 pad 2: GND -> /LED_GND1
- R34 pad 2: GND -> /LED_GND1
- R35 pad 2: GND -> /LED_GND1
- R36 pad 2: GND -> /LED_GND1
- SW1 pad 10: unconnected-(SW1-Pad10) -> GND
- SW1 pad 11: unconnected-(SW1-Pad11) -> GND
- SW1 pad 12: unconnected-(SW1-Pad12) -> GND
- SW1 pad 5: unconnected-(SW1-Pad5) -> /IN_GND0
- SW1 pad 6: unconnected-(SW1-Pad6) -> /IN_GND1
- SW1 pad 7: unconnected-(SW1-Pad7) -> /LED_GND0
- SW1 pad 8: unconnected-(SW1-Pad8) -> /LED_GND1
- SW1 pad 9: unconnected-(SW1-Pad9) -> GND
- SW2 pad 5: /IN4 -> /FPGA_CLK
- U3 pad 33: /SPI2_NSS -> /IN5
- U3 pad 56: /IN3 -> /IN2
- U3 pad 62: /BTN0 -> /IN3
- U4 pad 10: /IN4 -> /FPGA_CLK
- U4 pad 34: /SPI2_NSS -> /IN5
- U4 pad 36: /BTN1 -> /BTN0
- U4 pad 38: /BTN2 -> /BTN1

Commit message: did some placment
Parts:
- added C26: 100nF, PCM_JLCPCB:C_0603, F.Cu at (102.7, 90.7)
- added C27: 100nF, PCM_JLCPCB:C_0603, F.Cu at (116.7, 92.0)
- J10, J8, J9: footprint Connector_PinHeader_1.27mm:PinHeader_1x02_P1.27mm_Vertical -> Connector_PinHeader_2.54mm:PinHeader_1x02_P2.54mm_Vertical
- J11, J2: footprint Connector_PinHeader_1.27mm:PinHeader_1x06_P1.27mm_Vertical -> Connector_PinHeader_2.54mm:PinHeader_1x06_P2.54mm_Vertical
- J3: footprint Connector_PinHeader_1.27mm:PinHeader_1x16_P1.27mm_Vertical -> Connector_PinHeader_2.54mm:PinHeader_1x16_P2.54mm_Vertical
- J4, J5: footprint Connector_PinHeader_1.27mm:PinHeader_1x08_P1.27mm_Vertical -> Connector_PinHeader_2.54mm:PinHeader_1x08_P2.54mm_Vertical
- J6, J7: footprint Connector_PinHeader_1.27mm:PinHeader_1x03_P1.27mm_Vertical -> Connector_PinHeader_2.54mm:PinHeader_1x03_P2.54mm_Vertical
- moved J9 156.1 mm to (55.2, 29.8)
- moved R39 147.1 mm to (57.1, 71.2), turned to 90 degrees
- moved J6 144.7 mm to (83.2, 29.8)
- moved D13 142.4 mm to (57.1, 74.9), turned to -90 degrees
- moved C22 108.2 mm to (151.8, 51.8), turned to -90 degrees
- moved JP1 97.7 mm to (151.8, 48.3), turned to 90 degrees
- moved J8 92.3 mm to (168.9, 99.1)
- moved J7 89.7 mm to (168.3, 106.7)
- moved JP2 88.9 mm to (131.4, 89.5), turned to 90 degrees
- moved JP3 85.3 mm to (126.4, 89.5), turned to 90 degrees
- moved JP4 85.2 mm to (128.9, 89.5), turned to 90 degrees
- moved JP5 82.3 mm to (123.8, 89.5), turned to 90 degrees
- moved R38 79.5 mm to (117.6, 110.6), turned to 90 degrees
- moved R25 78.7 mm to (93.4, 114.5), turned to -90 degrees
- moved JP7 78.1 mm to (98.4, 109.4), turned to -90 degrees
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- renumbered C26 to C28, C28 to C29, C29 to C30, C30 to C31, R40 to R15, R42 to R16, R15 to R17, R16 to R18, R17 to R19, R18 to R20, R19 to R21, R20 to R22, R21 to R23, R22 to R24, R23 to R25, R24 to R26, R25 to R27, R26 to R28, R27 to R29, R28 to R30, R29 to R31, R30 to R32, R31 to R33, R32 to R34, R33 to R35, R34 to R36, R35 to R37, R36 to R38, R37 to R39, R38 to R40, R39 to R41, R41 to R42, R45 to R44, R47 to R45, R48 to R46, R49 to R47, S6 to S4
Connections:
- J5 pad 5: /FPGA_CLK -> /IN4
- JP4 pad 2: /FPGA_SPI_SO -> /FPGA_SPI_SI
- JP5 pad 2: /FPGA_SPI_SI -> /FPGA_SPI_SO
- R22 pad 2: /FPGA_CLK -> /IN4
- SW2 pad 5: /FPGA_CLK -> /IN4
- U3 pad 33: /IN5 -> /SPI2_NSS
- U4 pad 10: /FPGA_CLK -> /IN4
- U4 pad 34: /IN5 -> /SPI2_NSS
Routing:
- net +3V3: track 0.00 -> 22.4 mm, vias 0 -> 1
- net /FPGA_GLOBAL_1: track 0.00 -> 19.2 mm
- net /FPGA_CLK: track 0.00 -> 17.2 mm
- net GND: track 0.00 -> 16.6 mm, vias 0 -> 2
- net /SPI2_MOSI: track 0.00 -> 13.1 mm
- net /USART1_TX: track 0.00 -> 11.5 mm
- net /USART1_RX: track 0.00 -> 11.5 mm
- net /SPI2_NSS: track 0.00 -> 11.2 mm
- net /SPI2_SCK: track 0.00 -> 11.1 mm
- net /SPI2_MISO: track 0.00 -> 11.1 mm
- net /FPGA_USB_D+: track 0.00 -> 8.18 mm
- net /FPGA_USB_D-: track 0.00 -> 7.74 mm
- net /OSC_IN: track 0.00 -> 7.07 mm
- net +1V2: track 0.00 -> 6.34 mm, vias 0 -> 1
- net /VCCPLL: track 0.00 -> 4.88 mm, vias 0 -> 1
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Other:
- board size 70 x 70 mm -> 80 x 80 mm
- copper layers 2 -> 4
- board text added: "CDONE"
- board text added: "GND"
- board text added: "IN0"
- board text added: "IN1"
- board text added: "IN2"
- board text added: "IN3"
- board text added: "IN4"
- board text added: "IN5"
- board text added: "IN6"
- board text added: "IN7"
- board text added: "NRST"
- board text added: "OUT0"
- board text added: "OUT1"
- board text added: "OUT2"
- board text added: "OUT3"
- board text added: "OUT4"
- board text added: "OUT5"
- board text added: "OUT6"
- board text added: "OUT7"
- board text added: "PC0"
- board text added: "PC1"
- board text added: "PC10"
- board text added: "PC11"
- board text added: "PC12"
- board text added: "PC13"
- board text added: "PC14"
- board text added: "PC15"
- board text added: "PC2"
- board text added: "PC3"
- board text added: "PC4"
- board text added: "PC5"
- board text added: "PC6"
- board text added: "PC7"
- board text added: "PC8"
- board text added: "SWCLK"
- board text added: "SWDIO"
- board text added: "SWO"
- board text removed: "FPGA"

Commit message: lets push
Parts:
- removed the R17 at (118.9, 73.0)
- added R27: 68Ω, PCM_JLCPCB:R_0603, F.Cu at (118.7, 73.0)
- moved J9 71.1 mm to (64.8, 100.3)
- moved J6 63.1 mm to (64.8, 90.2), turned to 180 degrees
- moved C5 57.3 mm to (106.2, 79.5), turned to 180 degrees
- moved R6 55.8 mm to (128.8, 113.5)
- moved R5 55.2 mm to (127.2, 113.5)
- moved D4 54.6 mm to (123.2, 117.5)
- moved D1 54.5 mm to (125.7, 117.5)
- moved D2 54.5 mm to (128.3, 117.5)
- moved Q1 54.5 mm to (125.8, 109.5)
- moved R1 54.5 mm to (125.8, 106.5)
- moved R2 54.5 mm to (125.8, 113.5)
- moved C22 54.5 mm to (106.2, 81.8), turned to 180 degrees
- moved D3 54.5 mm to (130.8, 117.5)
- moved R30 53.9 mm to (124.2, 113.5)
- moved JP1 53.3 mm to (109.5, 80.8)
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- renumbered R18 to R17, R19 to R18, R20 to R19, R21 to R20, R22 to R21, R23 to R22, R24 to R23, R25 to R24, R26 to R25, R27 to R26
Connections:
- R25 pad 2: /FUD- -> /FPGA_USB_D-
Routing:
- net /IN5: track 0.00 -> 64.7 mm, vias 0 -> 1
- net /IN4: track 0.00 -> 63.4 mm, vias 0 -> 1
- net /IN7: track 0.00 -> 62.4 mm, vias 0 -> 1
- net /IN6: track 0.00 -> 62.0 mm, vias 0 -> 1
- net GND: track 16.6 -> 64.9 mm, vias 2 -> 12
- net /NRST: track 0.00 -> 46.5 mm, vias 0 -> 1
- net /PC0: track 0.00 -> 45.5 mm
- net +3V3: track 22.4 -> 66.8 mm, vias 1 -> 7
- net /I2C1_SCL: track 0.00 -> 43.6 mm, vias 0 -> 2
- net /I2C1_SDA: track 0.00 -> 43.4 mm, vias 0 -> 2
- net /PC1: track 0.00 -> 41.6 mm
- net /SWDIO: track 0.00 -> 37.1 mm, vias 0 -> 1
- net /PC2: track 0.00 -> 36.0 mm, vias 0 -> 1
- net /SWCLK: track 0.00 -> 34.7 mm, vias 0 -> 1
- net /PC6: track 2.43 -> 36.5 mm
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Other:
- board size 80 x 80 mm -> 80 x 70 mm
- board text added: "0"
- board text added: "1"
- board text added: "2"
- board text added: "BOOT0"
- board text added: "BOOT1"
- board text added: "BTN0"
- board text added: "BTN1"
- board text added: "CK"
- board text added: "CS"
- board text added: "FBOOT"
- board text added: "FPGA"
- board text added: "F_CS"
- board text added: "G3"
- board text added: "G6"
- board text added: "I2C"
- board text added: "I2S"
- board text added: "IN [0,3]"
- board text added: "IN [4,7]"
- board text added: "OUT [0,3]"
- board text added: "OUT [4,7]"
- board text added: "OUT8"
- board text added: "RESET FPGA"
- board text added: "RGB"
- board text added: "RX"
- board text added: "SCK"
- board text added: "SCL"
- board text added: "SD"
- board text added: "SDA"
- board text added: "SI"
- board text added: "SO"
- board text added: "TX"
- board text added: "UART"
- board text added: "WS"

Commit message: cleared up a bit
Parts:
- removed D10, D11, D12, D9: Green, PCM_JLCPCB:D_0805
- removed J4, J5: Conn_01x08_Pin, Connector_PinHeader_2.54mm:PinHeader_1x08_P2.54mm_Vertical
- removed JP12, JP13, JP6, JP7: SolderJumper_2_Open, Jumper:SolderJumper-2_P1.3mm_Open_RoundedPad1.0x1.5mm
- removed R21, R22, R23, R24: 15kΩ, PCM_JLCPCB:R_0603
- removed R35, R36, R37, R38: 1.5kΩ, PCM_JLCPCB:R_0603
- removed SW2: SW_DIP_x08, Button_Switch_THT:SW_DIP_SPSTx08_Slide_6.7x21.88mm_W7.62mm_P2.54mm_LowProfile
- moved R32 73.3 mm to (80.9, 168.2)
- moved D5 73.3 mm to (83.5, 172.0)
- moved D6 73.3 mm to (81.0, 172.0)
- moved D7 73.3 mm to (78.5, 172.0)
- moved D8 73.3 mm to (75.9, 172.0)
- moved R31 73.3 mm to (83.4, 168.2)
- moved R33 73.3 mm to (78.4, 168.2)
- moved R34 73.3 mm to (76.1, 168.2)
- moved D13 69.5 mm to (68.5, 171.1)
- moved R39 69.5 mm to (68.5, 167.8)
- moved R20 62.4 mm to (110.8, 50.2), turned to 90 degrees
- moved J2 61.8 mm to (30.5, 114.9)
- moved J3 61.8 mm to (30.5, 168.2)
- moved R19 60.9 mm to (108.5, 50.2), turned to 90 degrees
- moved R18 59.8 mm to (106.2, 50.2), turned to 90 degrees
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Connections:
- net /OUT8 renamed /OUT_STM
- R17 pad 1: /IN_GND0 -> GND
- R18 pad 1: /IN_GND0 -> GND
- R19 pad 1: /IN_GND0 -> GND
- R20 pad 1: /IN_GND0 -> GND
- R31 pad 2: /LED_GND0 -> GND
- R32 pad 2: /LED_GND0 -> GND
- R33 pad 2: /LED_GND0 -> GND
- R34 pad 2: /LED_GND0 -> GND
- SW1 pad 10: GND -> +3V3
- SW1 pad 11: GND -> +3V3
- SW1 pad 12: GND -> +3V3
- SW1 pad 5: /IN_GND0 -> /IN0
- SW1 pad 6: /IN_GND1 -> /IN1
- SW1 pad 7: /LED_GND0 -> /IN2
- SW1 pad 8: /LED_GND1 -> /IN3
- SW1 pad 9: GND -> +3V3
- U3 pad 14: /IN0 -> unconnected-(U3-PA0-Pad14)
- U3 pad 15: /IN1 -> unconnected-(U3-PA1-Pad15)
- U3 pad 56: /IN2 -> unconnected-(U3-PB4-Pad56)
- U3 pad 62: /IN3 -> unconnected-(U3-PB9-Pad62)
- U4 pad 10: /IN4 -> unconnected-(U4B-IOB_18a-Pad10)
- U4 pad 11: /IN5 -> unconnected-(U4B-IOB_20a-Pad11)
- U4 pad 4: /IN7 -> unconnected-(U4C-IOB_8a-Pad4)
- U4 pad 42: /OUT7 -> unconnected-(U4A-IOT_51a-Pad42)
- U4 pad 43: /OUT6 -> unconnected-(U4A-IOT_49a-Pad43)
- U4 pad 45: /OUT5 -> unconnected-(U4C-IOB_5b-Pad45)
- U4 pad 46: /OUT4 -> unconnected-(U4C-IOB_0a-Pad46)
- U4 pad 6: /IN6 -> unconnected-(U4B-IOB_13b-Pad6)
Routing:
- net +3V3: track 66.8 -> 0.00 mm, vias 7 -> 0
- net GND: track 64.9 -> 0.00 mm, vias 12 -> 0
- net /IN5: track 64.7 -> 0.00 mm, vias 1 -> 0
- net /IN4: track 63.4 -> 0.00 mm, vias 1 -> 0
- net /IN7: track 62.4 -> 0.00 mm, vias 1 -> 0
- net /IN6: track 62.0 -> 0.00 mm, vias 1 -> 0
- net /NRST: track 46.5 -> 0.00 mm, vias 1 -> 0
- net /PC0: track 45.5 -> 0.00 mm
- net /I2C1_SCL: track 43.6 -> 0.00 mm, vias 2 -> 0
- net /I2C1_SDA: track 43.4 -> 0.00 mm, vias 2 -> 0
- net /PC1: track 41.6 -> 0.00 mm
- net /SWDIO: track 37.1 -> 0.00 mm, vias 1 -> 0
- net /PC6: track 36.5 -> 0.00 mm, vias 1 -> 0
- net /PC7: track 36.1 -> 0.00 mm, vias 1 -> 0
- net /PC2: track 36.0 -> 0.00 mm, vias 1 -> 0
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Other:
- board text removed: "IN [0,3]"
- board text removed: "IN [4,7]"
- board text removed: "IN4"
- board text removed: "IN5"
- board text removed: "IN6"
- board text removed: "IN7"
- board text removed: "OUT [0,3]"
- board text removed: "OUT [4,7]"
- board text removed: "OUT4"
- board text removed: "OUT5"
- board text removed: "OUT6"
- board text removed: "OUT7"
