File: iCEBrainstorm/iCEBrainstorm.kicad_pcb (KiCad board)
At the start: 4 copper layers, 80 x 70 mm, 130 parts, among them J1 Connector, USB-TYPE-C-16P, J10 Conn_01x03_Pin, J11 Conn_01x04_Pin, J12 Conn_01x02_Pin, J13 Conn_01x02_Pin, J14 Conn_01x02_Pin, J15 Conn_01x06_Pin, J16 Connector, USB-TYPE-C-16P, J2 Conn_01x16_Pin, J3 Conn_01x06_Pin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

Commit message: send to production, note that the SM6DS3TR got replaced with the LSM6DSRTR for cost reasons.
Parts:
- moved PN1 81.4 mm to (96.5, 123.2), turned to -90 degrees
